Commit message: model update

File: robot_description/src/description/f1tenth_tt02.urdf (robot description, URDF)
Before this commit: robot racecar, 8 links, 7 joints
Links:
- added link base_vehicle; visual box size=${wheelbase} ${width} ${height}
- added link computer; visual box size=${wheelbase/2} ${width} ${computer_height}
- added link front_bumper; visual box size=${front_bumper} ${width} ${bumper_height}
- added link rear_bumper; visual box size=${rear_bumper} ${width} ${bumper_height}
- link base_link: geometry 
Joints:
- added joint base_link_to_base_vehicle: type fixed, parent base_link, child base_vehicle, origin rpy=0 0 3.1416
- added joint base_vehicle_to_computer: type fixed, parent base_vehicle, child computer, origin xyz=${wheelbase/4} 0 ${ground_offset+height+(computer_height/2)}
- added joint base_vehicle_to_front_bumper: type fixed, parent base_vehicle, child front_bumper, origin xyz=${(wheelbase)+(front_bumper/2)} 0 ${ground_offset+(bumper_height/2)}
- added joint base_vehicle_to_rear_bumper: type fixed, parent base_vehicle, child rear_bumper, origin xyz=${-(rear_bumper/2)} 0 ${ground_offset+(bumper_height/2)}
- joint base_to_back_left_wheel: parent base_link -> base_vehicle
- joint base_to_back_right_wheel: parent base_link -> base_vehicle
- joint base_to_front_left_hinge: parent base_link -> base_vehicle
- joint base_to_front_right_hinge: parent base_link -> base_vehicle
- joint base_to_laser: origin xyz=${laser_distance_from_base_link} 0 ${ground_offset+height+(laser_height/2)} -> xyz=${laser_distance_from_base_vehicle} 0 ${ground_offset+height+(laser_height/2)+laser_offset} rpy=0 0 3.1416; parent base_link -> base_vehicle
- joint front_left_hinge_to_wheel: type continuous -> fixed
- joint front_right_hinge_to_wheel: type continuous -> fixed
